Commit message: feat(sim): make the URDF physically valid and add a Gazebo Harmonic world
The description was visualisation-only: no inertials on half the links, no
collisions, no simulation plugins, and a geometry error that RViz could not
reveal.

Mechanical fix
--------------
The drive wheels were mounted at -base_height/2 relative to base_link, which
sits at +wheel_radius above base_footprint. Wheel centres therefore landed at
z=0 with a 0.06 m radius, putting the tyres 6 cm below the ground plane. It
looked correct in RViz only because there is no floor there; in a physics
engine the robot spawns buried.

Wheel joints are now at z=0 relative to base_link, so each centre sits at
exactly wheel_radius. A two-wheel box also has nowhere to rest, so front and
rear caster spheres were added, sized to the 3 cm ground clearance. Verified
from the generated URDF: all four contact points touch z=0.000 exactly.

Every link now carries an inertial block computed by a xacro macro rather
than the hand-written approximations, and collisions were added where they
were missing -- Gazebo silently drops links with neither.

Simulation layer
----------------
astro_gazebo.xacro holds everything simulation-specific and is included only
under sim_mode:=true, so the real robot's tf tree is untouched. It provides
DiffDrive (odom and odom->base_footprint tf), JointStatePublisher, a
JointPositionController for the head, and gpu_lidar / imu / camera sensors
matched to the real hardware: RPLIDAR A1 at 720 samples over 360 degrees,
0.15-12 m, and the OAK-D publishing to /oak/rgb/image_raw so the vision
nodes need no changes under simulation.

Plugin filenames target gz-sim 8; Gazebo Classic and Fortress names differ
and would fail silently here.

astro_sim package
-----------------
An indoor world -- corridor, three rooms with 0.9 m doorways, and furniture
that gives scan matching something to work with -- plus a launch file that
starts Gazebo, robot_state_publisher, the spawn, the ros_gz bridge and RViz.

Verified by running it headless: robot settles at z=0.000 with zero roll and
pitch, LiDAR returns 717 finite ranges out of 720 between 1.41 and 11.99 m,
and commanding 0.3 m/s moves odom 1.414 m forward with y unchanged. The tf
chain odom -> base_footprint -> laser_frame resolves, with the laser at
[0.100, 0, 0.110] from base_link.

Co-Authored-By: Claude Opus 5 <noreply@anthropic.com>

File: ros2_ws/src/astro_description/urdf/astro.urdf.xacro (robot description, xacro)
@@ -1,11 +1,72 @@
 <?xml version="1.0"?>
+<!--
+  ASTRO V1 — gövde tanımı (URDF/xacro)
+  Bu dosya hem gerçek robotta (yalnızca tf2 + RViz) hem de Gazebo Harmonic
+  simülasyonunda kullanılır. Simülasyona özgü her şey (eklentiler, sensörler,
+  sürtünme) ayrı astro_gazebo.xacro dosyasındadır ve YALNIZCA sim_mode:=true
+  iken dahil edilir; böylece gerçek robotun tf ağacı hiç değişmez.
+  Ölçü referansı: base_footprint zemindedir (z=0). Tekerlek merkezleri
+  z = wheel_radius olmak ZORUNDA, aksi hâlde robot fizik motorunda zemine
+  gömülür. Eski sürümde tekerlek eklemi base_link'e göre -base_height/2
+  konumundaydı ve merkez z=0'a düşüyordu: tekerlekler zeminin 6 cm altında
+  kalıyordu. RViz'de zemin düzlemi olmadığı için bu hata görünmüyordu.
+-->
 <robot xmlns:xacro="http://www.ros.org/wiki/xacro" name="astro">
-  <xacro:property name="base_length" value="0.30"/>
-  <xacro:property name="base_width" value="0.25"/>
-  <xacro:property name="base_height" value="0.12"/>
-  <xacro:property name="wheel_radius" value="0.06"/>
-  <xacro:property name="wheel_width" value="0.04"/>
+  <!-- true iken Gazebo eklentileri/sensörleri eklenir -->
+  <xacro:arg name="sim_mode" default="false"/>
+  <!-- ─────────────────────────── Ölçüler ─────────────────────────── -->
+  <xacro:property name="base_length"    value="0.30"/>
+  <xacro:property name="base_width"     value="0.25"/>
+  <xacro:property name="base_height"    value="0.12"/>
+  <xacro:property name="wheel_radius"   value="0.06"/>
+  <xacro:property name="wheel_width"    value="0.04"/>
   <xacro:property name="wheel_y_offset" value="0.13"/>
+  <xacro:property name="wheel_separation" value="${2 * wheel_y_offset}"/>
+  <!-- Zemin açıklığı: gövde alt yüzeyi ile zemin arası -->
+  <xacro:property name="ground_clearance" value="0.03"/>
+  <xacro:property name="caster_radius"     value="${ground_clearance}"/>
+  <xacro:property name="caster_x_offset"   value="0.11"/>
+  <!-- Gövde merkezinin base_link'e göre yüksekliği -->
+  <xacro:property name="body_z" value="${ground_clearance + base_height/2 - wheel_radius}"/>
   <xacro:property name="head_height" value="0.18"/>
+  <!-- ───────────────────── Atalet yardımcıları ───────────────────── -->
+  <!-- Gazebo kütlesiz/ataletsiz linkleri sessizce atar; her linkin
+       <inertial> bloğu olmak zorunda. -->
+  <xacro:macro name="inertial_box" params="mass x y z *origin">
+    <inertial>
+      <xacro:insert_block name="origin"/>
+      <mass value="${mass}"/>
+      <inertia ixx="${mass*(y*y+z*z)/12}" ixy="0" ixz="0"
+               iyy="${mass*(x*x+z*z)/12}" iyz="0"
+               izz="${mass*(x*x+y*y)/12}"/>
+    </inertial>
+  </xacro:macro>
+  <xacro:macro name="inertial_cylinder" params="mass radius length *origin">
+    <inertial>
+      <xacro:insert_block name="origin"/>
+      <mass value="${mass}"/>
+      <inertia ixx="${mass*(3*radius*radius+length*length)/12}" ixy="0" ixz="0"
+               iyy="${mass*(3*radius*radius+length*length)/12}" iyz="0"
+               izz="${mass*radius*radius/2}"/>
+    </inertial>
+  </xacro:macro>
+  <xacro:macro name="inertial_sphere" params="mass radius *origin">
+    <inertial>
+      <xacro:insert_block name="origin"/>
+      <mass value="${mass}"/>
+      <inertia ixx="${2*mass*radius*radius/5}" ixy="0" ixz="0"
+               iyy="${2*mass*radius*radius/5}" iyz="0"
+               izz="${2*mass*radius*radius/5}"/>
+    </inertial>
+  </xacro:macro>
+  <!-- ──────────────────────── Malzemeler ─────────────────────────── -->
+  <material name="grey">      <color rgba="0.5 0.5 0.5 1.0"/></material>
+  <material name="black">     <color rgba="0.1 0.1 0.1 1.0"/></material>
+  <material name="red">       <color rgba="0.8 0.1 0.1 1.0"/></material>
+  <material name="blue">      <color rgba="0.2 0.2 0.8 1.0"/></material>
+  <material name="white">     <color rgba="0.9 0.9 0.9 1.0"/></material>
+  <material name="dark_grey"> <color rgba="0.2 0.2 0.2 1.0"/></material>
+  <material name="green">     <color rgba="0.1 0.6 0.1 1.0"/></material>
+  <!-- ═══════════════════════ Taban ═══════════════════════ -->
   <link name="base_footprint"/>
   <joint name="base_footprint_joint" type="fixed">
@@ -16,134 +77,129 @@
   <link name="base_link">
     <visual>
-      <origin xyz="0 0 ${base_height/2}" rpy="0 0 0"/>
-      <geometry>
-        <box size="${base_length} ${base_width} ${base_height}"/>
-      </geometry>
-      <material name="grey">
-        <color rgba="0.5 0.5 0.5 1.0"/>
-      </material>
-    </visual>
-    <collision>
-      <origin xyz="0 0 ${base_height/2}" rpy="0 0 0"/>
-      <geometry>
-        <box size="${base_length} ${base_width} ${base_height}"/>
-      </geometry>
-    </collision>
-    <inertial>
-      <origin xyz="0 0 ${base_height/2}" rpy="0 0 0"/>
-      <mass value="5.0"/>
-      <inertia ixx="0.05" ixy="0" ixz="0" iyy="0.08" iyz="0" izz="0.1"/>
-    </inertial>
-  </link>
-  <link name="left_wheel_link">
-    <visual>
-      <geometry>
-        <cylinder radius="${wheel_radius}" length="${wheel_width}"/>
-      </geometry>
-      <material name="black">
-        <color rgba="0.1 0.1 0.1 1.0"/>
-      </material>
-    </visual>
-    <collision>
-      <geometry>
-        <cylinder radius="${wheel_radius}" length="${wheel_width}"/>
-      </geometry>
-    </collision>
-    <inertial>
-      <mass value="0.5"/>
-      <inertia ixx="0.001" ixy="0" ixz="0" iyy="0.001" iyz="0" izz="0.001"/>
-    </inertial>
-  </link>
-  <joint name="left_wheel_joint" type="continuous">
-    <parent link="base_link"/>
-    <child link="left_wheel_link"/>
-    <origin xyz="0 ${wheel_y_offset} ${-base_height/2}" rpy="1.5708 0 0"/>
-    <axis xyz="0 0 1"/>
-  </joint>
-  <link name="right_wheel_link">
-    <visual>
-      <geometry>
-        <cylinder radius="${wheel_radius}" length="${wheel_width}"/>
-      </geometry>
-      <material name="black">
-        <color rgba="0.1 0.1 0.1 1.0"/>
-      </material>
-    </visual>
-    <collision>
-      <geometry>
-        <cylinder radius="${wheel_radius}" length="${wheel_width}"/>
-      </geometry>
-    </collision>
-    <inertial>
-      <mass value="0.5"/>
-      <inertia ixx="0.001" ixy="0" ixz="0" iyy="0.001" iyz="0" izz="0.001"/>
-    </inertial>
-  </link>
-  <joint name="right_wheel_joint" type="continuous">
-    <parent link="base_link"/>
-    <child link="right_wheel_link"/>
-    <origin xyz="0 ${-wheel_y_offset} ${-base_height/2}" rpy="1.5708 0 0"/>
-    <axis xyz="0 0 1"/>
-  </joint>
+      <origin xyz="0 0 ${body_z}" rpy="0 0 0"/>
+      <geometry><box size="${base_length} ${base_width} ${base_height}"/></geometry>
+      <material name="grey"/>
+    </visual>
+    <collision>
+      <origin xyz="0 0 ${body_z}" rpy="0 0 0"/>
+      <geometry><box size="${base_length} ${base_width} ${base_height}"/></geometry>
+    </collision>
+    <xacro:inertial_box mass="5.0" x="${base_length}" y="${base_width}" z="${base_height}">
+      <origin xyz="0 0 ${body_z}" rpy="0 0 0"/>
+    </xacro:inertial_box>
+  </link>
+  <!-- ═══════════════════ Tahrik tekerlekleri ═══════════════════ -->
+  <!-- Eklem z=0: tekerlek merkezi base_footprint'ten wheel_radius yükseklikte,
+       yani lastik tam olarak zemine değiyor. -->
+  <xacro:macro name="drive_wheel" params="prefix y_sign">
+    <link name="${prefix}_wheel_link">
+      <visual>
+        <geometry><cylinder radius="${wheel_radius}" length="${wheel_width}"/></geometry>
+        <material name="black"/>
+      </visual>
+      <collision>
+        <geometry><cylinder radius="${wheel_radius}" length="${wheel_width}"/></geometry>
+      </collision>
+      <xacro:inertial_cylinder mass="0.5" radius="${wheel_radius}" length="${wheel_width}">
+        <origin xyz="0 0 0" rpy="0 0 0"/>
+      </xacro:inertial_cylinder>
+    </link>
+    <joint name="${prefix}_wheel_joint" type="continuous">
+      <parent link="base_link"/>
+      <child link="${prefix}_wheel_link"/>
+      <origin xyz="0 ${y_sign * wheel_y_offset} 0" rpy="${-pi/2} 0 0"/>
+      <axis xyz="0 0 1"/>
+      <dynamics damping="0.05" friction="0.02"/>
+    </joint>
+  </xacro:macro>
+  <xacro:drive_wheel prefix="left"  y_sign="1"/>
+  <xacro:drive_wheel prefix="right" y_sign="-1"/>
+  <!-- ═══════════════════ Denge tekerlekleri ═══════════════════ -->
+  <!-- İki tahrik tekerleği tek başına devrilir; ön ve arkaya birer küre
+       konuyor. Küre merkezi z = caster_radius olacak şekilde yerleştirilir. -->
+  <xacro:macro name="caster" params="prefix x_sign">
+    <link name="${prefix}_caster_link">
+      <visual>
+        <geometry><sphere radius="${caster_radius}"/></geometry>
+        <material name="dark_grey"/>
+      </visual>
+      <collision>
+        <geometry><sphere radius="${caster_radius}"/></geometry>
+      </collision>
+      <xacro:inertial_sphere mass="0.15" radius="${caster_radius}">
+        <origin xyz="0 0 0" rpy="0 0 0"/>
+      </xacro:inertial_sphere>
+    </link>
+    <joint name="${prefix}_caster_joint" type="fixed">
+      <parent link="base_link"/>
+      <child link="${prefix}_caster_link"/>
+      <origin xyz="${x_sign * caster_x_offset} 0 ${caster_radius - wheel_radius}" rpy="0 0 0"/>
+    </joint>
+  </xacro:macro>
+  <xacro:caster prefix="front" x_sign="1"/>
+  <xacro:caster prefix="rear"  x_sign="-1"/>
+  <!-- ═══════════════════════ IMU ═══════════════════════ -->
   <link name="imu_link">
-    <inertial>
-      <mass value="0.01"/>
-      <inertia ixx="0.00001" ixy="0" ixz="0" iyy="0.00001" iyz="0" izz="0.00001"/>
-    </inertial>
+    <xacro:inertial_box mass="0.01" x="0.02" y="0.02" z="0.005">
+      <origin xyz="0 0 0" rpy="0 0 0"/>
+    </xacro:inertial_box>
   </link>
   <joint name="imu_joint" type="fixed">
     <parent link="base_link"/>
     <child link="imu_link"/>
-    <origin xyz="0 0 ${base_height/2}" rpy="0 0 0"/>
-  </joint>
+    <origin xyz="0 0 ${body_z}" rpy="0 0 0"/>
+  </joint>
+  <!-- ═══════════════════════ LiDAR ═══════════════════════ -->
+  <!-- RPLIDAR A1: gövdenin üst yüzeyine, hafif öne monte -->
+  <xacro:property name="body_top" value="${body_z + base_height/2}"/>
   <link name="laser_frame">
     <visual>
-      <geometry>
-        <cylinder radius="0.04" length="0.04"/>
-      </geometry>
-      <material name="red">
-        <color rgba="0.8 0.1 0.1 1.0"/>
-      </material>
-    </visual>
+      <geometry><cylinder radius="0.04" length="0.04"/></geometry>
+      <material name="red"/>
+    </visual>
+    <collision>
+      <geometry><cylinder radius="0.04" length="0.04"/></geometry>
+    </collision>
+    <xacro:inertial_cylinder mass="0.17" radius="0.04" length="0.04">
+      <origin xyz="0 0 0" rpy="0 0 0"/>
+    </xacro:inertial_cylinder>
   </link>
   <joint name="laser_joint" type="fixed">
     <parent link="base_link"/>
     <child link="laser_frame"/>
-    <origin xyz="0.10 0 ${base_height + 0.02}" rpy="0 0 0"/>
-  </joint>
+    <origin xyz="0.10 0 ${body_top + 0.02}" rpy="0 0 0"/>
+  </joint>
+  <!-- ═══════════════════════ Kafa ═══════════════════════ -->
   <link name="head_yaw_link">
     <visual>
-      <geometry>
-        <cylinder radius="0.04" length="0.06"/>
-      </geometry>
-      <material name="blue">
-        <color rgba="0.2 0.2 0.8 1.0"/>
-      </material>
-    </visual>
-    <inertial>
-      <mass value="0.3"/>
-      <inertia ixx="0.001" ixy="0" ixz="0" iyy="0.001" iyz="0" izz="0.001"/>
-    </inertial>
+      <geometry><cylinder radius="0.04" length="0.06"/></geometry>
+      <material name="blue"/>
+    </visual>
+    <collision>
+      <geometry><cylinder radius="0.04" length="0.06"/></geometry>
+    </collision>
+    <xacro:inertial_cylinder mass="0.3" radius="0.04" length="0.06">
+      <origin xyz="0 0 0" rpy="0 0 0"/>
+    </xacro:inertial_cylinder>
   </link>
   <joint name="head_yaw_joint" type="revolute">
     <parent link="base_link"/>
     <child link="head_yaw_link"/>
-    <origin xyz="0 0 ${base_height + 0.04}" rpy="0 0 0"/>
+    <origin xyz="0 0 ${body_top + 0.03}" rpy="0 0 0"/>
     <axis xyz="0 0 1"/>
-    <limit lower="-1.57" upper="1.57" effort="1.0" velocity="1.0"/>
+    <limit lower="${-pi/2}" upper="${pi/2}" effort="1.0" velocity="1.0"/>
+    <dynamics damping="0.1" friction="0.05"/>
   </joint>
   <link name="head_link">
     <visual>
-      <geometry>
-        <box size="0.12 0.10 0.14"/>
-      </geometry>
-      <material name="white">
-        <color rgba="0.9 0.9 0.9 1.0"/>
-      </material>
-    </visual>
-    <inertial>
-      <mass value="0.5"/>
-      <inertia ixx="0.002" ixy="0" ixz="0" iyy="0.002" iyz="0" izz="0.002"/>
-    </inertial>
+      <geometry><box size="0.12 0.10 0.14"/></geometry>
+      <material name="white"/>
+    </visual>
+    <collision>
+      <geometry><box size="0.12 0.10 0.14"/></geometry>
+    </collision>
+    <xacro:inertial_box mass="0.5" x="0.12" y="0.10" z="0.14">
+      <origin xyz="0 0 0" rpy="0 0 0"/>
+    </xacro:inertial_box>
   </link>
   <joint name="head_pitch_joint" type="fixed">
@@ -152,13 +208,16 @@
     <origin xyz="0 0 ${head_height/2 + 0.03}" rpy="0 0 0"/>
   </joint>
+  <!-- ═══════════════════ OAK-D Lite kamera ═══════════════════ -->
   <link name="oak_link">
     <visual>
-      <geometry>
-        <box size="0.09 0.025 0.025"/>
-      </geometry>
-      <material name="dark_grey">
-        <color rgba="0.2 0.2 0.2 1.0"/>
-      </material>
-    </visual>
+      <geometry><box size="0.09 0.025 0.025"/></geometry>
+      <material name="dark_grey"/>
+    </visual>
+    <collision>
+      <geometry><box size="0.09 0.025 0.025"/></geometry>
+    </collision>
+    <xacro:inertial_box mass="0.06" x="0.09" y="0.025" z="0.025">
+      <origin xyz="0 0 0" rpy="0 0 0"/>
+    </xacro:inertial_box>
   </link>
   <joint name="oak_joint" type="fixed">
@@ -167,19 +226,23 @@
     <origin xyz="0.06 0 0.02" rpy="0 0 0"/>
   </joint>
+  <!-- Optik çerçeve: REP-103 (z ileri, x sağ, y aşağı) -->
   <link name="oak_rgb_camera_optical_frame"/>
   <joint name="oak_rgb_optical_joint" type="fixed">
     <parent link="oak_link"/>
     <child link="oak_rgb_camera_optical_frame"/>
-    <origin xyz="0 0 0" rpy="-1.5708 0 -1.5708"/>
-  </joint>
+    <origin xyz="0 0 0" rpy="${-pi/2} 0 ${-pi/2}"/>
+  </joint>
+  <!-- ═══════════════ ReSpeaker mikrofon dizisi ═══════════════ -->
   <link name="mic_link">
     <visual>
-      <geometry>
-        <cylinder radius="0.035" length="0.01"/>
-      </geometry>
-      <material name="green">
-        <color rgba="0.1 0.6 0.1 1.0"/>
-      </material>
-    </visual>
+      <geometry><cylinder radius="0.035" length="0.01"/></geometry>
+      <material name="green"/>
+    </visual>
+    <collision>
+      <geometry><cylinder radius="0.035" length="0.01"/></geometry>
+    </collision>
+    <xacro:inertial_cylinder mass="0.05" radius="0.035" length="0.01">
+      <origin xyz="0 0 0" rpy="0 0 0"/>
+    </xacro:inertial_cylinder>
   </link>
   <joint name="mic_joint" type="fixed">
@@ -188,3 +251,7 @@
     <origin xyz="0 0 ${head_height/2 + 0.01}" rpy="0 0 0"/>
   </joint>
+  <!-- ═══════════════ Simülasyon eklentileri ═══════════════ -->
+  <xacro:if value="$(arg sim_mode)">
+    <xacro:include filename="$(find astro_description)/urdf/astro_gazebo.xacro"/>
+  </xacro:if>
 </robot>
