Commit message: fix(sim): model casters as swivel wheels, add the mapped test world
In-place rotation was reading 14% off in odometry. Two friction values were
tried on the fixed caster spheres and the error changed sign rather than
shrinking:

  caster mu   straight    arc distance   arc heading   spin error
  0.02          --          +11.5%         -22.8 deg    -29.3 deg
  0.2          -0.8%         +5.2%          -1.3 deg    +22.2 deg

At mu=0.02 the chassis outruns the wheels when the drive stops, because
frictionless spheres let it coast round; at mu=0.2 the spheres resist and
the drive wheels slip instead. A sign flip means the error is kinematic, not
a friction coefficient waiting to be tuned: a fixed sphere has to scrub
sideways through every turn, which a caster does not.

Replaced with real swivel casters -- a vertical swivel joint plus a rolling
wheel whose contact trails 15 mm behind the swivel axis, so it self-aligns
with the direction of travel and never scrubs:

  swivel caster -2.7%         -0.8%          +2.4 deg    +14.0 deg

Arc heading error dropped from 22.8 deg to 2.4 deg and arc distance is now
within 1%. The residual on a pure in-place spin is the drive wheels' own
lateral scrub, which is physical and present on the real robot too.

Measured with the robot in clear corridor space. An earlier run put it at
(6.0, -3.5), which is inside the 0.22 m pillar at (6.0, -3.2), and the
readings from that run were meaningless.

Also adds the map produced by driving the test route: walls land within
1-4 cm of ground truth, inside the 5 cm cell size. After a ~35 m loop the
SLAM pose was 5 mm and 0.04 deg from the Gazebo pose, while map->odom shows
SLAM had absorbed 4.2 m and 17 deg of accumulated odometry error.

Co-Authored-By: Claude Opus 5 <noreply@anthropic.com>

File: ros2_ws/src/astro_description/urdf/astro.urdf.xacro (robot description, xacro)
@@ -115,24 +115,57 @@
   <xacro:drive_wheel prefix="left"  y_sign="1"/>
   <xacro:drive_wheel prefix="right" y_sign="-1"/>
-  <!-- ═══════════════════ Denge tekerlekleri ═══════════════════ -->
-  <!-- İki tahrik tekerleği tek başına devrilir; ön ve arkaya birer küre
-       konuyor. Küre merkezi z = caster_radius olacak şekilde yerleştirilir. -->
+  <!-- ═══════════════════ Döner denge tekerlekleri ═══════════════════ -->
+  <!--
+    İki tahrik tekerleği tek başına devrilir. Önce sabit küre denendi, ama
+    sabit küre yanlış model: sürtünmesi düşük olursa (mu=0.02) gövde yerinde
+    dönüşte ataletle kayıp odometriyi %14 aşıyor, yüksek olursa (mu=0.2) küre
+    direnip tahrik tekerleklerini patinaja sokuyor ve bu kez odometri %14
+    fazla okuyor. İşaretin tersine dönmesi, hatanın sürtünme katsayısında
+    değil kinematikte olduğunu gösterdi.
+    Gerçek robotta olduğu gibi döner teker: dikey döndürme ekseni + yuvarlanan
+    tekerlek, tekerlek teması döndürme ekseninin TRAIL kadar arkasında.
+    Bu geometri tekerleğin hareket yönüne kendiliğinden hizalanmasını sağlar
+    ve sürtünerek sürüklenme (scrub) tamamen ortadan kalkar.
+  -->
+  <xacro:property name="caster_trail" value="0.015"/>
   <xacro:macro name="caster" params="prefix x_sign">
-    <link name="${prefix}_caster_link">
+    <!-- Döndürme (swivel) mili -->
+    <link name="${prefix}_caster_swivel_link">
       <visual>
-        <geometry><sphere radius="${caster_radius}"/></geometry>
+        <geometry><cylinder radius="0.012" length="0.03"/></geometry>
         <material name="dark_grey"/>
       </visual>
+      <xacro:inertial_cylinder mass="0.03" radius="0.012" length="0.03">
+        <origin xyz="0 0 0" rpy="0 0 0"/>
+      </xacro:inertial_cylinder>
+    </link>
+    <joint name="${prefix}_caster_swivel_joint" type="continuous">
+      <parent link="base_link"/>
+      <child link="${prefix}_caster_swivel_link"/>
+      <origin xyz="${x_sign * caster_x_offset} 0 ${caster_radius - wheel_radius + 0.02}" rpy="0 0 0"/>
+      <axis xyz="0 0 1"/>
+      <dynamics damping="0.001" friction="0.0"/>
+    </joint>
+    <!-- Yuvarlanan tekerlek: milin TRAIL kadar arkasında -->
+    <link name="${prefix}_caster_wheel_link">
+      <visual>
+        <origin xyz="0 0 0" rpy="${pi/2} 0 0"/>
+        <geometry><cylinder radius="${caster_radius}" length="0.02"/></geometry>
+        <material name="black"/>
+      </visual>
       <collision>
-        <geometry><sphere radius="${caster_radius}"/></geometry>
+        <origin xyz="0 0 0" rpy="${pi/2} 0 0"/>
+        <geometry><cylinder radius="${caster_radius}" length="0.02"/></geometry>
       </collision>
-      <xacro:inertial_sphere mass="0.15" radius="${caster_radius}">
-        <origin xyz="0 0 0" rpy="0 0 0"/>
-      </xacro:inertial_sphere>
+      <xacro:inertial_cylinder mass="0.05" radius="${caster_radius}" length="0.02">
+        <origin xyz="0 0 0" rpy="${pi/2} 0 0"/>
+      </xacro:inertial_cylinder>
     </link>
-    <joint name="${prefix}_caster_joint" type="fixed">
-      <parent link="base_link"/>
-      <child link="${prefix}_caster_link"/>
-      <origin xyz="${x_sign * caster_x_offset} 0 ${caster_radius - wheel_radius}" rpy="0 0 0"/>
+    <joint name="${prefix}_caster_wheel_joint" type="continuous">
+      <parent link="${prefix}_caster_swivel_link"/>
+      <child link="${prefix}_caster_wheel_link"/>
+      <origin xyz="${-caster_trail} 0 -0.02" rpy="0 0 0"/>
+      <axis xyz="0 1 0"/>
+      <dynamics damping="0.001" friction="0.0"/>
     </joint>
   </xacro:macro>

File: ros2_ws/src/astro_description/urdf/astro_gazebo.xacro (robot description, xacro)
@@ -27,14 +27,16 @@
   <xacro:wheel_surface link="left_wheel_link"/>
   <xacro:wheel_surface link="right_wheel_link"/>
+  <!-- Döner teker artık yuvarlanıyor, sürüklenmiyor: gerçek lastik gibi
+       tutunabilir. Düşük sürtünmeye gerek yok. -->
   <xacro:macro name="caster_surface" params="link">
     <gazebo reference="${link}">
-      <mu1>0.02</mu1>
-      <mu2>0.02</mu2>
+      <mu1>0.8</mu1>
+      <mu2>0.8</mu2>
       <kp>1000000.0</kp>
       <kd>100.0</kd>
     </gazebo>
   </xacro:macro>
-  <xacro:caster_surface link="front_caster_link"/>
-  <xacro:caster_surface link="rear_caster_link"/>
+  <xacro:caster_surface link="front_caster_wheel_link"/>
+  <xacro:caster_surface link="rear_caster_wheel_link"/>
   <gazebo reference="base_link">
     <material>
@@ -74,4 +76,8 @@
       <joint_name>right_wheel_joint</joint_name>
       <joint_name>head_yaw_joint</joint_name>
+      <joint_name>front_caster_swivel_joint</joint_name>
+      <joint_name>front_caster_wheel_joint</joint_name>
+      <joint_name>rear_caster_swivel_joint</joint_name>
+      <joint_name>rear_caster_wheel_joint</joint_name>
     </plugin>
   </gazebo>
